Commit message: added collision and visual stls, have a loading ur20 with correct offsets

File: ur_description/urdf/inc/ur_common.xacro (robot description, xacro)
@@ -109,4 +109,7 @@
     <xacro:property name="shoulder_offset" value="${sec_offsets['shoulder_offset']}" scope="parent"/>
     <xacro:property name="elbow_offset" value="${sec_offsets['elbow_offset']}" scope="parent"/>
+    <xacro:property name="wrist_1_visual_offset" value="${sec_offsets['wrist_1_visual_offset']}" scope="parent"/>
+    <xacro:property name="wrist_2_visual_offset" value="${sec_offsets['wrist_2_visual_offset']}" scope="parent"/>
+    <xacro:property name="wrist_3_visual_offset" value="${sec_offsets['wrist_3_visual_offset']}" scope="parent"/>
     <!-- INERTIA PARAMETERS -->
     <!-- mass -->
@@ -180,5 +183,5 @@
     <xacro:property name="wrist_1_visual_material_color" value="${wrist_1_mesh['visual']['material']['color']}" scope="parent"/>
     <xacro:property name="wrist_1_collision_mesh" value="${wrist_1_mesh['collision']['mesh']}" scope="parent"/>
-    <xacro:property name="wrist_1_visual_offset" value="${wrist_1_mesh['visual_offset']}" scope="parent"/>
+    <!-- <xacro:property name="wrist_1_visual_offset" value="${wrist_1_mesh['visual_offset']}" scope="parent"/> -->
     <xacro:property name="wrist_2_mesh" value="${sec_mesh_files['wrist_2']}"/>
     <xacro:property name="wrist_2_visual_mesh" value="${wrist_2_mesh['visual']['mesh']}" scope="parent"/>
@@ -186,5 +189,5 @@
     <xacro:property name="wrist_2_visual_material_color" value="${wrist_2_mesh['visual']['material']['color']}" scope="parent"/>
     <xacro:property name="wrist_2_collision_mesh" value="${wrist_2_mesh['collision']['mesh']}" scope="parent"/>
-    <xacro:property name="wrist_2_visual_offset" value="${wrist_2_mesh['visual_offset']}" scope="parent"/>
+    <!-- <xacro:property name="wrist_2_visual_offset" value="${wrist_2_mesh['visual_offset']}" scope="parent"/> -->
     <xacro:property name="wrist_3_mesh" value="${sec_mesh_files['wrist_3']}"/>
     <xacro:property name="wrist_3_visual_mesh" value="${wrist_3_mesh['visual']['mesh']}" scope="parent"/>
@@ -192,5 +195,5 @@
     <xacro:property name="wrist_3_visual_material_color" value="${wrist_3_mesh['visual']['material']['color']}" scope="parent"/>
     <xacro:property name="wrist_3_collision_mesh" value="${wrist_3_mesh['collision']['mesh']}" scope="parent"/>
-    <xacro:property name="wrist_3_visual_offset" value="${wrist_3_mesh['visual_offset']}" scope="parent"/>
+    <!-- <xacro:property name="wrist_3_visual_offset" value="${wrist_3_mesh['visual_offset']}" scope="parent"/> -->
   </xacro:macro>
 </robot>

File: ur_description/urdf/inc/ur_macro.xacro (robot description, xacro)
@@ -63,4 +63,8 @@
     <!-- Add URDF transmission elements (for ros_control) -->
     <xacro:ur_arm_transmission prefix="${prefix}" hw_interface="${transmission_hw_interface}" />
+    <!-- Adding variables for unparamarized offset values -->
+    <!-- <xacro:property name="wrist_1_visual_offset" value="0.0"/>
+    <xacro:property name="wrist_2_visual_offset" value="0.0"/>
+    <xacro:property name="wrist_3_visual_offset" value="0.0"/> -->
     <!-- links: main serial chain -->
     <link name="${prefix}base_link"/>
